Commit message: [EL] simple urdf example with 3 IMUs

File: imu3_description/model/imu.urdf.xacro (robot description, xacro)
@@ -10,7 +10,7 @@
 			<parent link="${parent}"/>
 			<child link="${name}_first_link_roll"/>
-					<axis xyz="1 0 0" />
-				<limit lower="${0}" upper="${2*pi}" effort="${effort}" velocity="${velocity}"/>
-			</joint>
+			<axis xyz="1 0 0" />
+			<limit lower="${0}" upper="${2*pi}" effort="${effort}" velocity="${velocity}"/>
+		</joint>
 		<link name="${name}_first_link_roll">
 		</link>
@@ -108,4 +108,4 @@
 			</visual>
 		</link>
-	</xacro:macro> <!-- end xacro for one IMU -->
+	</xacro:macro> <!-- end xacro for 3 IMU -->
 </robot>

File: imu3_description/robot/imu3_simple.urdf.xacro (robot description, xacro)
@@ -7,20 +7,4 @@
 	<xacro:include filename="$(find imu3_description)/model/imu.urdf.xacro"/>
 	<link name="world">
-		 <!-- <inertial>
-		 <mass value="1"/>
-            <inertia ixx="0.13" iyy="0.524" izz="0.539" ixy="0" ixz="0" iyz="0" />
-            </inertial>
-		<visual>
-			<origin xyz="0 0 0.25" rpy="0 0 0"/>
-			<geometry>
-				<box size="0.5 0.5 0.5"/>
-			</geometry> -->
-			<!-- <material name="LightGrey" /> -->
-		<!-- </visual>
-		<collision>
-                <geometry>
-				<box size="0.5 0.5 0.5"/>
-                </geometry>
-            </collision>   -->
 	</link>
 	<xacro:imu parent="world" name="imu" position="0 0 0" orientation="0 0 0" />
